File: JTAG_dongle.kicad_sch (KiCad schematic)
At the start: 0 parts

Commit message: first routing
Parts:
- added J1: 5V supply Enable, Connector_PinHeader_2.54mm:PinHeader_1x02_P2.54mm_Vertical, symbol Connector_Generic:Conn_01x02
- added J2: SeggerJlink connector, local_footprints:SeggerJlinkFemaleConn, symbol Connector_Generic:Conn_02x10_Odd_Even
- added J3: Conn_02x10_Odd_Even, Connector_PinHeader_2.54mm:PinHeader_2x10_P2.54mm_Vertical, symbol Connector_Generic:Conn_02x10_Odd_Even
- added J4: FTS-105-01-F-D, Connector_PinHeader_1.27mm:PinHeader_2x05_P1.27mm_Vertical, symbol Connector_Generic:Conn_02x05_Odd_Even
- added JP1, JP10, JP11, JP12, JP13, JP14, JP15, JP16, JP17, JP18, JP19, JP2, JP20, JP21, JP22, JP23, JP24, JP25, JP26, JP27, JP28, JP29, JP3, JP30, JP31, JP32, JP33, JP34, JP35, JP36, JP37, JP38, JP39, JP4, JP40, JP41, JP42, JP43, JP44, JP45, JP46, JP47, JP48, JP49, JP5, JP6, JP7, JP8, JP9: SolderJumper_2_Bridged, Jumper:SolderJumper-2_P1.3mm_Bridged_Pad1.0x1.5mm, symbol Jumper:SolderJumper_2_Bridged
Connections:
- new net: J3.4 (Pin_4), JP41.1 (A)
- new net: J2.5 (Pin_5), JP3.2 (B)
- new net: J2.15 (Pin_15), JP8.2 (B)
- new net: J3.19 (Pin_19), JP39.2 (B)
- new net: J2.12 (Pin_12), JP15.1 (A)
- new net: J3.7 (Pin_7), JP33.2 (B)
- new net: J3.18 (Pin_18), JP48.1 (A)
- new net: J3.15 (Pin_15), JP37.2 (B)
- new net: J2.10 (Pin_10), JP14.1 (A)
- new net: J3.8 (Pin_8), JP43.1 (A)
- new net: J3.2 (Pin_2), JP40.1 (A)
- new net: J2.3 (Pin_3), JP2.2 (B)
- new net: J2.11 (Pin_11), JP6.2 (B)
- new net: J2.4 (Pin_4), JP11.1 (A)
- new net: J4.8 (Pin_8), JP28.1 (A)
- new net: J2.16 (Pin_16), JP17.1 (A)
- new net: J2.8 (Pin_8), JP13.1 (A)
- new net: J4.1 (Pin_1), JP20.2 (B)
- new net: J4.10 (Pin_10), JP29.1 (A)
- new net: J4.2 (Pin_2), JP25.1 (A)
- new net: J4.3 (Pin_3), JP21.2 (B)
- new net: J4.4 (Pin_4), JP26.1 (A)
- new net: J4.5 (Pin_5), JP22.2 (B)
- new net: J4.6 (Pin_6), JP27.1 (A)
- new net: J2.17 (Pin_17), JP9.2 (B)
- new net: J2.18 (Pin_18), JP18.1 (A)
- new net: J3.16 (Pin_16), JP47.1 (A)
- new net: J3.9 (Pin_9), JP34.2 (B)
- new net: J2.14 (Pin_14), JP16.1 (A)
- new net: J3.6 (Pin_6), JP42.1 (A)
- new net: J3.1 (Pin_1), JP30.2 (B)
- new net: J1.1 (Pin_1), J2.19 (Pin_19)
- new net: J3.5 (Pin_5), JP32.2 (B)
- new net: J3.13 (Pin_13), JP36.2 (B)
- new net: J2.6 (Pin_6), JP12.1 (A)
- new net: J2.1 (Pin_1), JP1.2 (B)
- new net: J2.13 (Pin_13), JP7.2 (B)
- new net: J2.2 (Pin_2), JP10.1 (A)
- new net: J2.20 (Pin_20), JP19.1 (A)
- new net: J2.7 (Pin_7), JP4.2 (B)
- new net: J2.9 (Pin_9), JP5.2 (B)
- new net: J3.12 (Pin_12), JP45.1 (A)
- new net: J3.3 (Pin_3), JP31.2 (B)
- new net: J3.10 (Pin_10), JP44.1 (A)
- new net: J3.14 (Pin_14), JP46.1 (A)
- new net: J3.11 (Pin_11), JP35.2 (B)
- new net: J3.17 (Pin_17), JP38.2 (B)
- new net: J3.20 (Pin_20), JP49.1 (A)
- new net 5V_Supply: J1.2 (Pin_2), JP39.1 (A)
- new net GND: JP11.2 (B), JP12.2 (B), JP13.2 (B), JP14.2 (B), JP15.2 (B), JP21.1 (A), JP22.1 (A), JP24.1 (A), JP41.2 (B), JP42.2 (B), JP43.2 (B), JP44.2 (B), JP45.2 (B)
- new net GND_Detect: J4.9 (Pin_9), JP24.2 (B)
- new net KEY: J4.7 (Pin_7), JP23.2 (B)
- new net RESET: JP29.2 (B), JP37.1 (A), JP8.1 (A)
- new net RTCK: JP35.1 (A), JP6.1 (A)
- new net TCK/SWCLK: JP26.2 (B), JP34.1 (A), JP5.1 (A)
- new net TDI: JP28.2 (B), JP3.1 (A), JP32.1 (A)
- new net TDO/SWO: JP27.2 (B), JP36.1 (A), JP7.1 (A)
- new net TMS/SWDIO: JP25.2 (B), JP33.1 (A), JP4.1 (A)
- new net VTref: JP1.1 (A), JP20.1 (A), JP30.1 (A)
- new net nTRST: JP2.1 (A), JP31.1 (A)
- no-connect marks 0 -> 13
